File: AD8015/OneInchAD8015/OneInchAD8015.kicad_sch (KiCad schematic)
At the start: 37 parts, among them J1 Conn_01x03, J2 RF, U1 LT3042EMSE, U2 AD8015, U3 LM321

Commit message: pot for mon
Parts:
- removed R7: 100k, Resistor_SMD:R_0402_1005Metric, symbol Device:R
- added C11: 1n, Capacitor_SMD:C_0402_1005Metric, symbol Device:C
- added RV1: 100k, Potentiometer_SMD:Potentiometer_Bourns_TC33X_Vertical, symbol Device:R_Potentiometer_Trim
- D3, TP1, TP2: now not fitted
- J1: footprint Connector_PinHeader_2.54mm:PinHeader_1x03_P2.54mm_Vertical -> Connector_PinHeader_2.00mm:PinHeader_1x03_P2.00mm_Vertical; now not fitted
- R10: value 22k -> 10k; footprint Resistor_SMD:R_0603_1608Metric -> Resistor_SMD:R_0402_1005Metric; LCSC C31850 -> C25744
- R11: value 1k -> 1.5k; LCSC (none) -> C22843
- R2: value 2.2k -> 1.5k; LCSC (none) -> C22843
- U2: LCSC (none) -> C514255
- U3: LCSC (none) -> C471859
Connections:
- net GND: now also C11.1
- net at R6.2, U3.1 (+): now also C11.2
- net at R10.1, U3.3 (-): now also RV1.3
- net at J1.3 (Pin_3), R11.2, U3.4: now also RV1.1, RV1.2
