File: AD8015/OneInchAD8015/OneInchAD8015.kicad_pcb (KiCad board)
At the start: 2 copper layers, 25 x 25 mm, 37 parts, among them J1 Conn_01x03, J2 RF, U1 LT3042EMSE, U2 AD8015, U3 LM321

Commit message: labels
Routing:
- net GND: vias 0 -> 17
Other:
- board text added: "Mitchell A. Cox, 2025 github.com/WitsOCLab"
- board text added: "OneInchAD8015 v1.0"
Changed lines of the file:
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@@
 		)
+	)
+	(gr_rect
+		(start 104.3 93.4)
+		(end 109.2 106.5)
+		(stroke
+			(width 0.12)
+			(type solid)
+		)
+		(fill solid)
+		(layer "B.SilkS")
 	)
 	(gr_circle
@@
 	)
 	(gr_text "5.1V"
-		(at 109 98 0)
+		(at 110.4 98.5 90)
 		(layer "B.SilkS")
 		(effects
@@
 			)
 			(justify left bottom)
+		)
+	)
+	(gr_text "Mitchell A. Cox, 2025\ngithub.com/WitsOCLab"
+		(at 100 92.3 0)
+		(layer "B.Mask")
+		(effects
+			(font
+				(size 0.7 0.7)
+				(thickness 0.15)
+			)
+			(justify bottom mirror)
+		)
+	)
+	(gr_text "OneInchAD8015 v1.0"
+		(at 95.9 95.7 0)
+		(layer "B.Mask")
+		(effects
+			(font
+				(size 0.7 0.7)
+				(thickness 0.15)
+			)
+			(justify bottom mirror)
 		)
 	)
@@
 		(net 2)
 	)
+	(via
+		(at 100.9 89.6)
+		(size 0.8)
+		(drill 0.4)
+		(layers "F.Cu" "B.Cu")
+		(free yes)
+		(net 2)
+	)
+	(via
+		(at 107.75 107.65)
+		(size 0.8)
+		(drill 0.4)
+		(layers "F.Cu" "B.Cu")
+		(free yes)
+		(net 2)
+	)
+	(via
+		(at 92.7 91.9)
+		(size 0.8)
+		(drill 0.4)
+		(layers "F.Cu" "B.Cu")
+		(free yes)
+		(net 2)
+	)
+	(via
+		(at 92.5 106.8)
+		(size 0.8)
+		(drill 0.4)
+		(layers "F.Cu" "B.Cu")
+		(free yes)
+		(net 2)
+	)
+	(via
+		(at 108.8 102.8)
+		(size 0.8)
+		(drill 0.4)
+		(layers "F.Cu" "B.Cu")
+		(free yes)
+		(net 2)
+	)
+	(via
+		(at 107 96.5)
+		(size 0.8)
+		(drill 0.4)
+		(layers "F.Cu" "B.Cu")
+		(free yes)
+		(net 2)
+	)
+	(via
+		(at 107 101.3)
+		(size 0.8)
+		(drill 0.4)
+		(layers "F.Cu" "B.Cu")
+		(free yes)
+		(net 2)
+	)
+	(via
+		(at 98.2 95)
+		(size 0.8)
+		(drill 0.4)
+		(layers "F.Cu" "B.Cu")
+		(free yes)
+		(net 2)
+	)
+	(via
+		(at 97.4 106.9)
+		(size 0.8)
+		(drill 0.4)
+		(layers "F.Cu" "B.Cu")
+		(free yes)
+		(net 2)
+	)
+	(via
+		(at 102.65 104)
+		(size 0.8)
+		(drill 0.4)
+		(layers "F.Cu" "B.Cu")
+		(free yes)
+		(net 2)
+	)
+	(via
+		(at 99.1 89.6)
+		(size 0.8)
+		(drill 0.4)
+		(layers "F.Cu" "B.Cu")
+		(free yes)
+		(net 2)
+	)
+	(via
+		(at 105 102.8)
+		(size 0.8)
+		(drill 0.4)
+		(layers "F.Cu" "B.Cu")
+		(free yes)
+		(net 2)
+	)
+	(via
+		(at 92.55 102.05)
+		(size 0.8)
+		(drill 0.4)
+		(layers "F.Cu" "B.Cu")
+		(free yes)
+		(net 2)
+	)
+	(via
+		(at 95.85 96.25)
+		(size 0.8)
+		(drill 0.4)
+		(layers "F.Cu" "B.Cu")
+		(free yes)
+		(net 2)
+	)
+	(via
+		(at 110.9 101.35)
+		(size 0.8)
+		(drill 0.4)
+		(layers "F.Cu" "B.Cu")
+		(free yes)
+		(net 2)
+	)
+	(via
+		(at 106.9 92.6)
+		(size 0.8)
+		(drill 0.4)
+		(layers "F.Cu" "B.Cu")
+		(free yes)
+		(net 2)
+	)
+	(via
+		(at 95.4 94.5)
+		(size 0.8)
+		(drill 0.4)
+		(layers "F.Cu" "B.Cu")
+		(free yes)
+		(net 2)
+	)

Commit message: pot for mon
Parts:
- removed the R8 at (93.8, 105.9)
- removed the R9 at (95.2, 105.9)
- added C11: 1n, Capacitor_SMD:C_0402_1005Metric, F.Cu at (100.2, 104.5)
- added R10: 10k, Resistor_SMD:R_0402_1005Metric, F.Cu at (94.8, 108.2)
- added RV1: 100k, Potentiometer_SMD:Potentiometer_Bourns_TC33X_Vertical, F.Cu at (93.1, 105.6)
- J1: footprint Connector_PinHeader_2.54mm:PinHeader_1x03_P2.54mm_Vertical -> Connector_PinHeader_2.00mm:PinHeader_1x03_P2.00mm_Vertical
- R11: value 1k -> 1.5k
- R2: renamed from R1; value 2.2k -> 1.5k
- moved R11 1.52 mm to (96.4, 109.8)
- moved R6 0.90 mm to (102.0, 104.5)
- moved C4 0.15 mm to (98.5, 108.9)
- moved C7 0.11 mm to (95.8, 99.4)
- moved D1 0.10 mm to (94.7, 101.3)
- moved D4 0.10 mm to (100.3, 110.7)
- moved R8 0.10 mm to (94.7, 103.0)
- moved U3 0.10 mm to (97.5, 105.9)
- renumbered C2 to C1, C3 to C12, C9 to C13, C11 to C14, C4 to C2, C1 to C3, C13 to C4, C6 to C5, C5 to C6, C8 to C7, C7 to C8, C12 to C9, D3 to D1, D1 to D2, D2 to D3, L2 to L1, L1 to L2, R3 to R1, R4 to R3, R5 to R4, R10 to R5, R7 to R6, R6 to R8, R2 to R9
Routing:
- net Net-(J1-Pin_3): track 9.59 -> 15.2 mm
- net Net-(U3--): track 3.48 -> 5.70 mm
- net Net-(U3-+): track 2.57 -> 4.29 mm
- net Net-(D4-A): track 4.25 -> 2.58 mm
- net GND: vias 17 -> 16
Other:
- board text added: "M"
- board text added: "V+"
- board text removed: "Rf"
- board text removed: "Rg"

Commit message: mods
Parts:
- added D5: LED, LED_SMD:LED_0603_1608Metric, B.Cu at (100.0, 104.1)
- C7: value 10n -> 100n
- moved D1 1.24 mm to (93.8, 102.1), turned to 90 degrees
- moved R8 1.10 mm to (95.5, 102.2), turned to 90 degrees
- moved C8 0.20 mm to (105.0, 97.7)
- moved C7 0.15 mm to (95.8, 99.5), turned to -90 degrees
- moved C14 0.10 mm to (103.8, 103.4)
- turned R4 to 90 degrees
Routing:
- net Net-(D4-A): track 2.58 -> 9.29 mm, vias 0 -> 1
- net Net-(L2-Pad1): track 9.67 -> 8.02 mm
- net Net-(D3-A): track 5.68 -> 6.78 mm
- net GND: track 4.57 -> 5.47 mm, vias 16 -> 20
- net /+9V: track 22.9 -> 22.3 mm
