File: MAX40658/OneInchMAX/OneInchMAX.kicad_sch (KiCad schematic)
At the start: 39 parts, among them J1 Conn_01x03, J2 RF, U1 LT3042EMSE, U2 AD8015, U3 LM321

Commit message: mods
Parts:
- removed R4: 10k, Resistor_SMD:R_0402_1005Metric, symbol Device:R
- removed R5: 49.9, Resistor_SMD:R_0402_1005Metric, symbol Device:R
- removed R8: 10, Resistor_SMD:R_0603_1608Metric, symbol Device:R
- removed U2: AD8015, Package_SO:SOIC-8_3.9x4.9mm_P1.27mm, symbol Amplifier_Operational:AD8015
- added C15, C16: 1n C0G, Capacitor_SMD:C_0402_1005Metric, symbol Device:C
- added R12, R7: 49.9, Resistor_SMD:R_0402_1005Metric, symbol Device:R
- added R13, R14: 75, Resistor_SMD:R_0402_1005Metric, symbol Device:R
- added TP3: OFFSET, TestPoint:TestPoint_THTPad_D1.0mm_Drill0.5mm, symbol Connector:TestPoint
- added U2: MAX40658, Package_DFN_QFN:TDFN-8_1.4x1.6mm_P0.4mm, symbol MAX40658:MAX40658
- added U4: BUF602xDBV, Package_TO_SOT_SMD:SOT-23-5, symbol Amplifier_Buffer:BUF602xDBV
- C10: value 100n -> 1n C0G; JLCPCB C1525 -> C76947; LCSC C1525 -> C76947
- C13: value 10n -> 1u; JLCPCB C15195 -> (none); LCSC C15195 -> C29266
- C14: value 100n -> 1u; JLCPCB C1525 -> (none); LCSC C1525 -> C29266
- C8: value 10n C0G -> 1n C0G; footprint Capacitor_SMD:C_0603_1608Metric -> Capacitor_SMD:C_0402_1005Metric; JLCPCB C76710 -> C76947; LCSC C76710 -> C76947
Connections:
- net GND: now also C14.1, C15.1, R12.2, R13.2, R14.2, U2.5 (GND), U2.8 (GND), U4.2 (V-); no longer C14.2
- net at R6.1: no longer J2.1 (In)
- net at C10.1, C6.3, C9.1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: now also C7.1, U2.1 (+V), U4.5 (V+)
- net at L2.1: now also D1.1 (K)
- net at C8.1, D3.3 (A): now also R12.1
- net at C13.1: now also U2.3 (CCAP); no longer C14.1
- net at C8.2: now also U2.2 (Iin)
- net at C5.3, D3.1 (K): now also C15.2; no longer C7.1
- new net: C14.2, R7.1, U2.4 (OFFSET)
- new net: C16.1, U4.1
- new net: R13.1, U2.6 (+), U4.4 (IN)
- new net: R14.1, U2.7 (-)
- new net: R7.2, TP3.1
- new net: C16.2, J2.1 (In)
Other:
- note removed: "MMCX connector Digikey WM5557-ND"
- moved on the sheet: C11, C4, D4, D5, J2, R10, R11, R6, RV1, U3
