File: OPA818_TwoInch/oip_opa818.kicad_pcb (KiCad board)
At the start: 2 copper layers, 50 x 50 mm, 47 parts, among them J1 Conn_Coaxial, J101 Conn_Coaxial, J102 Conn_01x03, U1 AD8656, U101 LT3042xMSE, U102 LT3093xMSE, U103 OPA818IDRGx, U104 BUF602xDBV

Commit message: v1 for jlc
Parts:
- C104: footprint Capacitor_SMD:C_0603_1608Metric -> Capacitor_SMD:C_0402_1005Metric
- C115: value C -> 0.6p
- C3: value 10n -> 1n
- R106: value 49R9 -> 49.9R
- R2: value 21.2k -> 16k
- R3: value 1.28k -> 16k
- RF101: value R -> 1.2k

Commit message: v1 of OneInchAD8015
Parts:
- removed C6, C7: NFM21PC105B1C3D, NFM:NFM21C
- removed D101, D103: D, Diode_SMD:D_SOD-323F
- removed J102: Conn_01x03, Connector_PinHeader_2.54mm:PinHeader_1x03_P2.54mm_Vertical
- added -9V1: TPM9, TestPoint:TestPoint_THTPad_D1.0mm_Drill0.5mm, F.Cu at (157.4, 101.8)
- added 9V1: TP9, TestPoint:TestPoint_THTPad_D1.0mm_Drill0.5mm, F.Cu at (155.9, 104.5)
- added C2: 22u, Capacitor_SMD:C_0805_2012Metric, F.Cu at (147.8, 119.2)
- added C8: 22u, Capacitor_SMD:C_0805_2012Metric, F.Cu at (165.1, 96.5)
- added C9: 22u, Capacitor_SMD:C_0805_2012Metric, F.Cu at (169.3, 96.5)
- added D3: D, Diode_SMD:D_SOD-323F, F.Cu at (144.8, 118.5)
- added D4: LED, LED_SMD:LED_0603_1608Metric, F.Cu at (167.1, 90.3)
- added D5: LED, LED_SMD:LED_0603_1608Metric, F.Cu at (163.2, 90.3)
- added GND1: TPGND, TestPoint:TestPoint_THTPad_D1.0mm_Drill0.5mm, F.Cu at (161.1, 92.2)
- added J4: ~, Connector_PinHeader_2.54mm:PinHeader_1x04_P2.54mm_Vertical, F.Cu at (145.4, 113.5)
- added L1: 10u, Inductor_SMD:L_0805_2012Metric, F.Cu at (149.9, 119.2)
- added L2: 10u, Inductor_SMD:L_0805_2012Metric, F.Cu at (167.4, 96.5)
- added L3: 10u, Inductor_SMD:L_0805_2012Metric, F.Cu at (163.2, 96.5)
- added PS1: WRA1209CS-3W, Converter_DCDC:Converter_DCDC_XP_POWER-ITQxxxxS-H_THT, F.Cu at (153.0, 115.5)
- added R10: 2.2k, Resistor_SMD:R_0402_1005Metric, F.Cu at (163.2, 92.9)
- added R7: 470, Resistor_SMD:R_0402_1005Metric, F.Cu at (136.2, 95.2)
- added R8: 2.2k, Resistor_SMD:R_0402_1005Metric, F.Cu at (167.1, 92.9)
- added R9: 2.2k, Resistor_SMD:R_0603_1608Metric, F.Cu at (135.0, 113.2)
- C115: value 0.6p -> 0.2p
- D1: footprint LED_SMD:LED_0201_0603Metric -> LED_SMD:LED_0603_1608Metric
- D2: footprint LED_SMD:LED_0201_0603Metric -> LED_THT:LED_D3.0mm_Clear
- J1: value Conn_Coaxial -> Monitor
- R5: footprint Resistor_SMD:R_0402_1005Metric -> Resistor_SMD:R_0603_1608Metric
- RF101: value 1.2k -> 5.1k
- moved D1 4.48 mm to (138.2, 94.5)
- moved D2 3.34 mm to (135.0, 89.9)
- moved J1 0.55 mm to (135.3, 108.5)
- moved R5 0.26 mm to (133.3, 104.5)
- moved C104 0.20 mm to (151.0, 104.0)
Connections:
- net Net-(D101-K) renamed /+9V
- net Net-(D103-A) renamed /-9V
- net Net-(J1-In) renamed INTENSITY
- D2 pad 2: Net-(D1-A) -> Net-(D2-A)
Routing:
- net /+9V: track 16.2 -> 47.6 mm
- net /-9V: track 21.3 -> 38.3 mm
- net Net-(PS1-+Vout): track 0.00 -> 14.3 mm, vias 0 -> 1
- net Net-(PS1-+Vin): track 0.00 -> 9.75 mm
- net /+VIN: track 9.02 -> 0.00 mm
- net /-VIN: track 8.32 -> 0.00 mm
- net INTENSITY: track 4.74 -> 12.0 mm
- net Net-(PS1--Vout): track 0.00 -> 6.39 mm, vias 0 -> 1
- net Net-(D2-A): track 0.00 -> 6.01 mm, vias 0 -> 1
- net Net-(D3-A): track 0.00 -> 5.71 mm
- net Net-(D3-K): track 0.00 -> 5.28 mm
- net Net-(J102-Pin_1): track 2.97 -> 0.00 mm
- net Net-(J102-Pin_3): track 2.92 -> 0.00 mm
- net Net-(D1-A): track 2.51 -> 5.33 mm, vias 1 -> 0
- net Net-(U1B--): track 2.26 -> 4.32 mm
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Other:
- board text added: "-9V"
- board text added: "."
- board text added: "9V"
- board text added: "IPD14"
- board text added: "MON"
- board text added: "MON = 5.1*R9/(R5+R9) < 10 kHz"
- board text added: "PDA"
- board text added: "PDC"
- board text removed: "-12V"
- board text removed: "Intensity"
- board text removed: "MONITOR < 10 kHz"

Commit message: seems to be done, ac coupled
Parts:
- removed C104: 10n, Capacitor_SMD:C_0402_1005Metric
- removed C105, C106, C108, C109: 100n, Capacitor_SMD:C_0603_1608Metric
- removed D1: LED, LED_SMD:LED_0603_1608Metric
- removed D2: LED, LED_THT:LED_D3.0mm_Clear
- removed J1: Monitor, Connector_Coaxial:MMCX_Molex_73415-1471_Vertical
- removed R2, R3: 16k, Resistor_SMD:R_0402_1005Metric
- removed R4: 100, Resistor_SMD:R_0402_1005Metric
- removed R5: 49.9R, Resistor_SMD:R_0603_1608Metric
- removed R6, R7: 470, Resistor_SMD:R_0402_1005Metric
- removed R9: 2.2k, Resistor_SMD:R_0603_1608Metric
- removed RF1: 0R, Resistor_SMD:R_0402_1005Metric
- added C10: 1n C0G, Capacitor_SMD:C_0402_1005Metric, F.Cu at (147.8, 96.0)
- added C11: 1n C0G, Capacitor_SMD:C_0402_1005Metric, B.Cu at (148.6, 98.4)
- added C12: 1n C0G, Capacitor_SMD:C_0402_1005Metric, F.Cu at (140.1, 103.2)
- added C13: 1n C0G, Capacitor_SMD:C_0402_1005Metric, F.Cu at (140.1, 100.5)
- added C14: 1n C0G, Capacitor_SMD:C_0402_1005Metric, F.Cu at (141.7, 94.6)
- added C15: 1n C0G, Capacitor_SMD:C_0402_1005Metric, F.Cu at (144.5, 97.6)
- added C16: 100n, Capacitor_SMD:C_0402_1005Metric, F.Cu at (141.4, 99.5)
- added C17: 1n C0G, Capacitor_SMD:C_0402_1005Metric, F.Cu at (134.0, 104.0)
- added C6: 10n, Capacitor_SMD:C_0402_1005Metric, F.Cu at (133.6, 95.5)
- added C7: 100n, Capacitor_SMD:C_0402_1005Metric, F.Cu at (141.7, 93.7)
- added D6: LED, LED_SMD:LED_0603_1608Metric, F.Cu at (138.4, 107.3)
- added D7: LED, LED_SMD:LED_0603_1608Metric, B.Cu at (153.3, 104.0)
- added H1: MountingHole, MountingHole:MountingHole_3.2mm_M3_DIN965_Pad_TopBottom, F.Cu at (157.5, 79.3)
- added H2: MountingHole, MountingHole:MountingHole_3.2mm_M3_DIN965_Pad_TopBottom, F.Cu at (128.3, 103.8)
- added H3: MountingHole, MountingHole:MountingHole_3.2mm_M3_DIN965_Pad_TopBottom, F.Cu at (164.1, 116.8)
- added Q1: BC857, Package_TO_SOT_SMD:SOT-323_SC-70, F.Cu at (148.8, 104.2)
- added R103: 300R, Resistor_SMD:R_0603_1608Metric, F.Cu at (151.4, 92.3)
- added R11: 100, Resistor_SMD:R_0402_1005Metric, F.Cu at (136.4, 100.5)
- added R15: 100, Resistor_SMD:R_0402_1005Metric, F.Cu at (151.1, 104.2)
- added R16: 100k, Resistor_SMD:R_0402_1005Metric, F.Cu at (138.4, 100.9)
- added R17: 10k, Resistor_SMD:R_0402_1005Metric, F.Cu at (136.9, 105.7)
- added R18: 1.5k, Resistor_SMD:R_0603_1608Metric, F.Cu at (139.2, 109.7)
- added R19: 100, Resistor_SMD:R_0402_1005Metric, F.Cu at (134.7, 95.5)
- added R20: 10k, Resistor_SMD:R_0402_1005Metric, F.Cu at (138.4, 99.7)
- added RV1: 100k, Potentiometer_SMD:Potentiometer_Bourns_TC33X_Vertical, F.Cu at (133.6, 107.2)
- C115: value 0.2p -> 0.1p
- C3, C4: value 1n -> 100n
- L101: value 100u -> 47uH
- moved J101 7.19 mm to (143.2, 90.2), turned to -90 degrees
- moved C5 5.90 mm to (145.4, 97.6)
- moved C4 3.59 mm to (139.1, 103.2), turned to -90 degrees
- moved C102 3.51 mm to (150.2, 94.0), turned to 0 degrees
- moved C3 3.33 mm to (135.9, 102.0), turned to -90 degrees
- moved R106 1.91 mm to (143.2, 93.7), turned to -90 degrees
- moved 9V1 1.06 mm to (157.0, 104.7)
- moved C112 0.84 mm to (154.8, 100.9)
- moved C113 0.84 mm to (160.1, 99.4)
- moved C114 0.84 mm to (156.0, 92.5)
- moved R102 0.84 mm to (153.9, 94.7)
- moved R107 0.84 mm to (160.1, 97.9)
- moved U102 0.84 mm to (156.8, 95.9)
- moved C101 0.30 mm to (151.2, 109.8)
- moved C107 0.30 mm to (148.2, 109.8)
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Connections:
- C3 pad 1: Net-(C3-Pad1) -> /-V
- C3 pad 2: Net-(U1A--) -> GND
- C4 pad 1: GND -> /+V
- C4 pad 2: Net-(U1A-+) -> GND
- C5 pad 1: Net-(U104-IN) -> GND
- C5 pad 2: Net-(C5-Pad2) -> /+V
- D5 pad 1: GND -> Net-(D5-K)
- D5 pad 2: Net-(D5-A) -> GND
- R10 pad 1: Net-(D5-A) -> Net-(D5-K)
- U1 pad 1: Net-(U1A--) -> INTENSITY
- U1 pad 4: GND -> /-V
- U1 pad 5: Net-(U1A--) -> GND
- U1 pad 7: Net-(U1B--) -> Net-(C6-Pad1)
- U104 pad 4: Net-(U104-IN) -> /VTIA
Routing:
- net /-V: track 34.1 -> 75.4 mm, vias 2 -> 3
- net /+V: track 57.7 -> 81.0 mm
- net Net-(D6-A): track 0.00 -> 20.8 mm, vias 0 -> 1
- net Net-(Q1-B): track 0.00 -> 17.5 mm, vias 0 -> 2
- net /-9V: track 38.3 -> 52.4 mm, vias 0 -> 1
- net Net-(C6-Pad1): track 0.00 -> 6.50 mm
- net Net-(D2-A): track 6.01 -> 0.00 mm, vias 1 -> 0
- net /VTIA: track 1.21 -> 7.21 mm
- net Net-(D1-A): track 5.33 -> 0.00 mm
- net /IN-: track 7.77 -> 13.0 mm
- net INTENSITY: track 12.0 -> 16.6 mm
- net Net-(L101-Pad1): track 1.35 -> 5.54 mm
- net GND: track 27.0 -> 23.2 mm, vias 86 -> 83
- net Net-(U1A--): track 10.3 -> 7.34 mm
- net Net-(U1B--): track 4.32 -> 7.20 mm
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Other:
- board text added: "-5V:"
- board text added: "Bias -9V:"
- board text added: "DC-couple"
- board text added: "Monitor Gain"
- board text added: "RF"
- board text added: "Remove for"
- board text added: "fc = 1.6 kHz"
- board text added: "github.com/WitsOCLab/Two-Inch-Photodetector Mitchell A. Cox 2025"
- board text removed: "+"
- board text removed: "-"
- board text removed: "IPD14"
- board text removed: "MON = 5.1*R9/(R5+R9) < 10 kHz"
- board text removed: "RF > 15 kHz"
- board text removed: "github.com/WitsOCLab/Two-Inch-Photodetector Mitchell A. Cox 2023"
