File: OPA818_TwoInch/oip_opa818.kicad_sch (KiCad schematic)
At the start: 47 parts, among them J1 Conn_Coaxial, J101 Conn_Coaxial, J102 Conn_01x03, U1 AD8656, U101 LT3042xMSE, U102 LT3093xMSE, U103 OPA818IDRGx, U104 BUF602xDBV

Commit message: v1 for jlc
Parts:
- C1, C5: JLCPCB (none) -> C307331; LCSC (none) -> C307331
- C101, C102, C103, C107, C112, C113, C114: JLCPCB (none) -> C19666; LCSC (none) -> C19666
- C104: footprint Capacitor_SMD:C_0603_1608Metric -> Capacitor_SMD:C_0402_1005Metric; JLCPCB (none) -> C15195; LCSC (none) -> C15195
- C105, C106, C108, C109: JLCPCB (none) -> C14663; LCSC (none) -> C14663
- C115: value C -> 0.6p; JLCPCB (none) -> C2857968; LCSC (none) -> C2857968
- C3: value 10n -> 1n; JLCPCB (none) -> C1523; LCSC (none) -> C1523
- C31: JLCPCB (none) -> C92518; LCSC (none) -> C92518
- C4: JLCPCB (none) -> C1523; LCSC (none) -> C1523
- D1, D2: JLCPCB (none) -> C2286; LCSC (none) -> C2286
- D101, D103: JLCPCB (none) -> C191023; LCSC (none) -> C191023
- J1, J101: JLCPCB (none) -> C530664; LCSC (none) -> C530664
- L101: JLCPCB (none) -> C68035; LCSC (none) -> C68035
- R1: JLCPCB (none) -> C25077; LCSC (none) -> C25077
- R101, R107: JLCPCB (none) -> C25794; LCSC (none) -> C25794
- R102: JLCPCB (none) -> C25102; LCSC (none) -> C25102
- R106: value 49R9 -> 49.9R; JLCPCB (none) -> C25120; LCSC (none) -> C25120
- R2: value 21.2k -> 16k; JLCPCB (none) -> C3015838; LCSC (none) -> C3015838
- R3: value 1.28k -> 16k; JLCPCB (none) -> C3015838; LCSC (none) -> C3015838
- R4: JLCPCB (none) -> C25076; LCSC (none) -> C25076
- R5: JLCPCB (none) -> C25120; LCSC (none) -> C25120
- R6: JLCPCB (none) -> C25117; LCSC (none) -> C25117
- RF1: JLCPCB (none) -> C17168; LCSC (none) -> C17168
- RF101: value R -> 1.2k; JLCPCB (none) -> C25862; LCSC (none) -> C25862
- U1: JLCPCB (none) -> C208582
- U101: JLCPCB (none) -> C461518; LCSC (none) -> C461518
- U102: JLCPCB (none) -> C670481; LCSC (none) -> C670481
- U103: JLCPCB (none) -> C2859543; LCSC (none) -> C2859543
- U104: JLCPCB (none) -> C2862949; LCSC (none) -> C2862949
Other:
- note added: "fc = 9.9 kHz (-3 dB) -20 dB @ 30 kHz"
- note removed: "fc = 10 kHz (-3 dB) (Chebyshev 0.02 dB) -0 dB @ 3 kHz -12.7 dB @ 20 kHz -28.6 dB @ 50 kHz"

Commit message: v1 of OneInchAD8015
Parts:
- removed C31 (x2): NFM21PC105B1C3D, NFM:NFM21C, symbol Device:Filter_EMI_C
- removed D101, D103: D, Diode_SMD:D_SOD-323F, symbol Device:D
- removed J102: Conn_01x03, Connector_PinHeader_2.54mm:PinHeader_1x03_P2.54mm_Vertical, symbol Connector_Generic:Conn_01x03
- added -9V1: TPM9, TestPoint:TestPoint_THTPad_D1.0mm_Drill0.5mm, symbol Connector:TestPoint
- added 9V1: TP9, TestPoint:TestPoint_THTPad_D1.0mm_Drill0.5mm, symbol Connector:TestPoint
- added C2, C8, C9: 22u, Capacitor_SMD:C_0805_2012Metric, symbol Device:C
- added C6: 2.2u, Capacitor_SMD:C_0402_1005Metric, symbol Device:C
- added C7: 4u7, Capacitor_SMD:C_0603_1608Metric, symbol Device:C
- added D3: D, Diode_SMD:D_SOD-323F, symbol Device:D
- added D4, D5: LED, LED_SMD:LED_0603_1608Metric, symbol Device:LED
- added GND1: TPGND, TestPoint:TestPoint_THTPad_D1.0mm_Drill0.5mm, symbol Connector:TestPoint
- added J4: ~, Connector_PinHeader_2.54mm:PinHeader_1x04_P2.54mm_Vertical, symbol Connector_Generic:Conn_01x04
- added L1, L2, L3: 10u, Inductor_SMD:L_0805_2012Metric, symbol Device:L
- added PS1: WRA1209CS-3W, Converter_DCDC:Converter_DCDC_XP_POWER-ITQxxxxS-H_THT, symbol Converter_DCDC:ITQ2415S
- added Q1: PMBT4403, Package_TO_SOT_SMD:SOT-23, symbol Device:Q_PNP_BEC
- added R10, R8: 2.2k, Resistor_SMD:R_0402_1005Metric, symbol Device:R
- added R11, R15: 100, Resistor_SMD:R_0402_1005Metric, symbol Device:R
- added R12: 1M, Resistor_SMD:R_0402_1005Metric, symbol Device:R
- added R13, R14: 100k, Resistor_SMD:R_0402_1005Metric, symbol Device:R
- added R7: 470, Resistor_SMD:R_0402_1005Metric, symbol Device:R
- added R9: 2.2k, Resistor_SMD:R_0603_1608Metric, symbol Device:R
- C115: value 0.6p -> 0.1p; JLCPCB C2857968 -> (none); LCSC C2857968 -> (none)
- D1: footprint LED_SMD:LED_0201_0603Metric -> LED_SMD:LED_0603_1608Metric; JLCPCB C2286 -> C72043; LCSC C2286 -> C72043
- D2: footprint LED_SMD:LED_0201_0603Metric -> LED_THT:LED_D3.0mm_Clear; JLCPCB C2286 -> C72043; LCSC C2286 -> C72043
- J1: value Conn_Coaxial -> Monitor
- R101, R107: JLCPCB C25794 -> C23186; LCSC C25794 -> C23186
- R102: JLCPCB C25102 -> C23025; LCSC C25102 -> C23025
- R5: footprint Resistor_SMD:R_0402_1005Metric -> Resistor_SMD:R_0603_1608Metric; JLCPCB C25120 -> C23185; LCSC C25120 -> C23185
- RF101: value 1.2k -> 5.1k; JLCPCB C25862 -> C351692; LCSC C25862 -> C351692
- U101: JLCPCB C461518 -> C69847; LCSC C461518 -> C69847
- U102: JLCPCB C670481 -> C670490; LCSC C670481 -> C670490
Connections:
- net +V: now also R13.1
- net GND: now also C2.2, C7.2, C8.2, C9.2, D4.1 (K), D5.2 (A), GND1.1, J4.2 (Pin_2), J4.3 (Pin_3), PS1.1 (-Vin), PS1.7 (Common), R14.2, R15.2, R9.2
- net IN-: now also Q1.3 (C)
- net +9V: now reaches C101.1, U101.1 (IN), U101.2 (IN), U101.3 (EN/UV), U101.6 (PGFB)
- net +9V: now also 9V1.1, C9.1, L2.2, R8.2
- net -9V: now reaches C112.2, U102.1 (IN), U102.13 (IN), U102.2 (IN), U102.3 (EN/UV), U102.5 (PGFB)
- net -9V: now also -9V1.1, C8.1, L3.2, R10.2
- net at C3.2, R5.2, U1.1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: no longer U1.5 (+)
- net at D1.2 (A), R6.1: no longer D2.2 (A)
- net INTENSITY: now reaches J1.1 (In), R5.1
- net INTENSITY: now also J4.4 (Pin_4), R9.1
- net at C5.2, R3.2, RF1.1: now also R12.1
- new net: Q1.2 (E), R15.1
- new net: C2.1, D3.1 (K), L1.1
- new net: D3.2 (A), J4.1 (Pin_1)
- new net: D4.2 (A), R8.1
- new net: C6.1, R11.1, U1.7
- new net: C6.2, R12.2, U1.6 (-)
- new net: D5.1 (K), R10.1
- new net: Q1.1 (B), R11.2
- new net: C7.1, R13.2, R14.1, U1.5 (+)
- new net: L2.1, PS1.6 (+Vout)
- new net: D2.2 (A), R7.1
- new net: L1.2, PS1.2 (+Vin)
- new net: L3.1, PS1.8 (-Vout)
- new net: R6.2, R7.2
Other:
- note removed: "Lead colors Brown (+12V) Black (GND) Blue (-12V)"
- note removed: "PSU: Thorlabs LDS12B ±12 VDC Regulated Linear Power Supply, 6 W Lumberg RSMV3 male connector, 3-pin PSU-lead: Digikey A120947-ND (mates with Thorlabs 3-pin psu connector) 3-pin M8 female connector 1.5 m 3-wire lead, solder to PCB"
- moved on the sheet: C1, C101, C103, C107, C112, C113, C114, R101, R107, TP101, TP102, U101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

Commit message: mods
Parts:
- removed C104: 10n, Capacitor_SMD:C_0402_1005Metric, symbol Device:C
- removed C4: 1n, Capacitor_SMD:C_0402_1005Metric, symbol Device:C
- removed C5: 100n, Capacitor_SMD:C_0402_1005Metric, symbol Device:C
- removed C7: 4u7, Capacitor_SMD:C_0603_1608Metric, symbol Device:C
- removed D1: LED, LED_SMD:LED_0603_1608Metric, symbol Device:LED
- removed D2: LED, LED_THT:LED_D3.0mm_Clear, symbol Device:LED
- removed R13, R14: 100k, Resistor_SMD:R_0402_1005Metric, symbol Device:R
- removed R2, R3: 16k, Resistor_SMD:R_0402_1005Metric, symbol Device:R
- removed R4: 100, Resistor_SMD:R_0402_1005Metric, symbol Device:R
- removed R5: 49.9R, Resistor_SMD:R_0603_1608Metric, symbol Device:R
- removed R6, R7: 470, Resistor_SMD:R_0402_1005Metric, symbol Device:R
- removed R9: 2.2k, Resistor_SMD:R_0603_1608Metric, symbol Device:R
- removed RF1: 0R, Resistor_SMD:R_0402_1005Metric, symbol Device:R
- added C10: 1n C0G, Capacitor_SMD:C_0402_1005Metric, symbol Device:C
- added C11: 1n, Capacitor_SMD:C_0402_1005Metric, symbol Device:C
- added D6, D7: LED, LED_SMD:LED_0603_1608Metric, symbol Device:LED
- added R16: 100k, Resistor_SMD:R_0402_1005Metric, symbol Device:R
- added R17: 10k, Resistor_SMD:R_0402_1005Metric, symbol Device:R
- added R18: 1.5k, Resistor_SMD:R_0603_1608Metric, symbol Device:R
- added R19: 100, Resistor_SMD:R_0402_1005Metric, symbol Device:R
- added RV1: 100k, Potentiometer_SMD:Potentiometer_Bourns_TC33X_Vertical, symbol Device:R_Potentiometer_Trim
- C3: value 1n -> 100n; JLCPCB C1523 -> C307331; LCSC C1523 -> C307331
Connections:
- net -5VBIAS: now also C10.1
- net -V: now also C3.1, U1.4 (V-)
- net GND: now also C3.2, U1.5 (+), C10.2, C11.1, D6.1 (K), D7.1 (K), R17.2; no longer U1.4 (V-)
- net INTENSITY: now also U1.1, R18.2, RV1.1, RV1.2
- net VTIA: now also R12.1, U104.4 (IN), R16.1
- net at R12.2, U1.6 (-): now also R19.1; no longer C6.2
- net at U1.3 (+): now also C11.2, R16.2
- new net: D6.2 (A), D7.2 (A), R18.1
- new net: C6.2, R19.2
- new net: R17.1, RV1.3, U1.2 (-)
Other:
- note added: "f_c = 1.6 kHz"
- note removed: "fc = 15 kHz"
- note removed: "fc = 9.9 kHz (-3 dB) -20 dB @ 30 kHz"
- moved on the sheet: C6

Commit message: seems to be done, ac coupled
Parts:
- removed C105, C106, C108, C109: 100n, Capacitor_SMD:C_0603_1608Metric, symbol Device:C
- removed J1: Monitor, Connector_Coaxial:MMCX_Molex_73415-1471_Vertical, symbol Connector:Conn_Coaxial
- removed R12: 1M, Resistor_SMD:R_0402_1005Metric, symbol Device:R
- added C12, C13, C14, C15, C17: 1n C0G, Capacitor_SMD:C_0402_1005Metric, symbol Device:C
- added C16, C4, C5, C7: 100n, Capacitor_SMD:C_0402_1005Metric, symbol Device:C
- added H1, H2, H3: MountingHole, MountingHole:MountingHole_3.2mm_M3_DIN965_Pad_TopBottom, symbol Mechanical:MountingHole
- added R103: 300R, Resistor_SMD:R_0603_1608Metric, symbol Device:R
- added R20: 10k, Resistor_SMD:R_0402_1005Metric, symbol Device:R
- C11: value 1n -> 1n C0G; JLCPCB (none) -> C76947; LCSC C1523 -> C76947
- C115: LCSC (none) -> C53273
- C6: value 2.2u -> 10n; LCSC (none) -> C15195
- L101: value 100u -> 47uH; JLCPCB C68035 -> (none); LCSC C68035 -> C404762
- Q1: value PMBT4403 -> BC857; footprint Package_TO_SOT_SMD:SOT-23 -> Package_TO_SOT_SMD:SOT-323_SC-70; LCSC C75556 -> C8660
- R18: JLCPCB C21190 -> (none)
Connections:
- net +V: now also C12.2, C15.2, C4.1, C5.2
- net -5VBIAS: now also C11.1
- net -9V: now also R103.1
- net -V: now also C13.1, C14.1, C16.1, C7.1
- net GND: now also C11.2, Q1.2 (E), C12.1, C13.2, C14.2, C15.1, C16.2, C17.2, C4.2, C5.1, C7.2; no longer C11.1, R15.2
- net IN-: now also R15.1; no longer Q1.3 (C)
- net VTIA: now also R20.2
- net at L101.1, R102.2: now also R103.2
- net at R16.2, U1.3 (+): now also C17.1; no longer C11.2
- net at R19.2: now also U1.6 (-), R20.1; no longer C6.2
- net at R19.1: now also C6.2; no longer U1.6 (-)
- new net: Q1.3 (C), R15.2
Other:
- note removed: "12" MMCX-to-SMA lead, RG316 Digikey 744-1700-ND"
- moved on the sheet: -9V1, 9V1, C1, C10, C101, C102, C103, C107, C112, C113, C114, C115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

Commit message: finished?
Parts:
- C115: value 0.1p -> 0.2p; LCSC C53273 -> C76908
Changed lines of the file:
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@@
+			"AAAAAAAAAAAAAAAAAAAAAAAAAAAAAAAAAAAAAAAAAAAAAAAAAAAAAAAAAAAAAAAAAAAAAAAAAAAA"
+			"AAAAAAAAAAAAAAAAAAAAAAAAAAAAAAAAAAAAAAAAAAAAAAAAAAAAAAAAAAAAAAAAAAAAAAAAAAAA"
+			"AAAAAAAAAAAAAAAAAAAAAAAAAAAAAAAAAAAAAAAAAAAAAAAAAAAAAAAAAAAAAAAAAAAAAAAAAAAA"
+			"AAAAAAAAAAAAAAAAAAAAAAAAAAAAAAAAAAAAAAAAAAAAAAAAAAAAAAAAAAAAAAAAAAAAAAAAAAAA"
+			"AAAAAAAAAAAAAAAAAAAAAAAAAAAAAAAAAAAAAAAAAAAAAAAAAAAAAAAAAAAAAAAAAAAAAAAAAAAA"
+			"AAAAAAAAAAAAAAAAAAAAAAAAAAAAAAAAAAAAAAAAAAAAAAAAAAAAAAAAAAAAAAAAAAAAAAAAAAAA"
+			"AAAAAAAAAAAAAAAAAAAAAAAAAAAAAAAAAAAAAAAAAAAAAAAAAAAAAAAAAAAAAAAAAAAAAAAAAAAA"
+			"AAAAAAAAAAAAAAAAAAAAAAAAAAAAAAAAAAAAAAAAAAAAAAAAAAAAAAAAAAAAAAAAAAAAAAAAAAAA"
+			"AAAAAAAAAAAAAAAAAAAAAAAAAAAAAAAAAAAAAAAAAAAAAAAAAAAAAAAAAAAAAAAAAAAAAAAAAAAA"
+			"AAAAAAAAAAAAAAAAAAAAAAAAAAAAAAAAAAAAAAAAAAAAAAAAAAAAAAAAAAAAAAAAAAAAAAAAAAAA"
+			"AAAAAAAAAAAAAAAAAAAAAAAAAAAAAAAAAAAAAAAAAAAAAAAAAAAAAAAAAAAAAAAAAAAAAAAAAAAA"
+			"AAAAAAAAAAAAAAAAAAAAAAAAAAAAAAAAAAAAAAAAAAAAAAAAAAAAAAAAAAAAAAAAAAAAAAAAAAAA"
+			"AAAAAAAAAAAAAAAAAAAAAAAAAAAAAAAAAAAAAAAAAAAAAAAAAAAAAAAAAAAAAAAAAAAAAAAAAAAA"
+			"AAAAAAAAAAAAAAAAAAAAAAAAAAAAAAAAAAAAAAAAAAAAAAAAAAAAAAAAAAAAAAAAAAAAAAAAAAAA"
+			"AAAAAAAAAAAAAAAAAAAAAAAAAAAAAAAAAAAAAAAAAAAAAAAAAAAAAAAAAAAAAAAAAAAAAAAAAAAA"
+			"AAAAAAAAAAAAAAAAAAAAAAAAAAAAAAAAAAAAAAAAAAAAAAAAAAAAAAAAAAAAAAAAAAAAAAAAAAAA"
+			"AAAAAAAAAAAAAAAAAAAAAAAAAAAAAAAAAAAAAAAAAAAAAAAAAAAAAAAAAAAAAAAAAAAAAAAAAAAA"
+			"AAAAAAAAAAAAAAAAAAAAAAAAAAAAAAAAAAAAAAAAAAAAAAAAAAAAAAAAAAAAAAAAAAAAAAAAAAAA"
+			"AAAAAAAAAAAAAAAAAAAAAAAAAAAAAAAAAAAAAAAAAAAAAAAAAAAAAAAAAAAAAAAAAAAAAAAAAAAA"
+			"AAAAAAAAAAAAAAAAAAAAAAAAAAAAAAAAAAAAAAAAAAAAAAAAAAAAAAAAAAAAAAAAAAAAAAAAAAAA"
+			"AAAAAAAAAAAAAAAAAAAAAAAAAAAAAAAAAAAAAAAAAAAAAAAAAAAAAAAAAAAAAAAAAAAAAAAAAAAA"
+			"AAAAAAAAAAAAAAAAAAAAAAAAAAAAAAAAAAAAAAAAAAAAAAAAAAAAAAAAAAAAAAAAAAAAAAAAAAAA"
+			"AAAAAAAAAAAAAAAAAAAAAAAAAAAAAAAAAAAAAAAAAAAAAAAAAAAAAAAAAAAAAAAAAAAAAAAAAAAA"
+			"AAAAAAAAAAAAAAAAAAAAAAAAAAAAAAAAAAAAAAAAAAAAAAAAAAAAAAAAAAAAAAAAAAAAAAAAAAAA"
+			"AAAAAAAAAAAAAAAAAAAAAAAAAAAAAAAAAAAAAAAAAAAAAAAAAAAAAAAAAAAAAAAAAAAAAAAAAAAA"
+			"AAAAAAAAAAAAAAAAAAAAAAAAAAAAAAAAAAAAAAAAAAAAAAAAAAAAAAAAAAAAAAAAAAAAAAAAAAAA"
+			"AAAAAAAAAAAAAAAAAAAAAAAAAAAAAAAAAAAAAAAAAAAAAAAAAAAAAAAAAAAAAAAAAAAAAAAAAAAA"
+			"AAAAAAAAAAAAAAAAAAAAAAAAAAAAAAAAAAAAAAAAAAAAAAAAAAAAAAAAAAAAAAAAAAAAAAAAAAAA"
+			"AAAAAAAAAAAAAAAAAAAAAAAAAAAAAAAAAAAAAAAAAAAAAAAAAAAAAAAAAAAAAAAAAAAAAAAAAAAA"
+			"AAAAAAAAAAAAAAAAAAAAAAAAAAAAAAAAAAAAAAAAAAAAAAAAAAAAAAAAAAAAAAAAAAAAAAAAAAAA"
+			"AAAAAAAAAAAAAAAAAAAAAAAAAAAAAAAAAAAAAAAAAAAAAAAAAAAAAAAAAAAAAAAAAAAAAAAAAAAA"
+			"AAAAAAAAAAAAAAAAAAAAAAAAAAAAAAAAAAAAAAAAAAAAAAAAAAAAAAAAAAAAAAAAAAAAAAAAAAAA"
+			"AAAAAAAAAAAAAAAAAAAAAAAAAAAAAAAAAAAAAAAAAAAAAAAAAAAAAAAAAAAAAAAAAAAAAAAAAAAA"
+			"AAAAAAAAAAAAAAAAAAAAAAAAAAAAAAAAAAAAAAAAAAAAAAAAAAAAAAAAAAAAAAAAAAAAAAAAAAAA"
+			"AAAAAAAAAAAAAAAAAAAAAAAAAAAAAAAAAAAAAAAAAAAAAAAAAAAAAAAAAAAAAAAAAAAAAAAAAAAA"
+			"AAAAAAAAAAAAAAAAAAAAAAAAAAAAAAAAAAAAAAAAAAAAAAAAAAAAAAAAAAAAAAAAAAAAAAAAAAAA"
 			"AAAAAAAAAAAAAAAAAAAAAAAAAAAAAAAAAAAAAAAAAAAAAAAAAAAAAAAAAAAAAAAAAAAAAAAAAAAA"
 			"AAAAAAAAAAAAAAAAAAAAAAAAAAAAAAAAAAAAAAAAAAAAAAAAAAAAAAAAAAAAAAAAAAAAAAAAAAAA"
@@
 			)
 		)
-		(property "Value" "0.1p"
+		(property "Value" "0.2p"
 			(at 162.56 46.99 0)
 			(effects
@@
 			)
 		)
-		(property "LCSC" "C53273"
+		(property "LCSC" "C76908"
 			(at 165.1 49.53 0)
 			(effects
